Commit message: E31

File: body.urdf (robot description, URDF)
Before this commit: robot robot, 2 links, 1 joints
Links:
- removed link Leg
- removed link Torso
- added link Link0, mass 1; collision box size=1 1 1; visual box size=1 1 1
- added link Link1, mass 1; collision box size=1 1 1; visual box size=1 1 1
Joints:
- removed joint Torso_Leg
- added joint Link0_Link1: type revolute, parent Link0, child Link1, origin xyz=0.5 0 1 rpy=0 0 0, axis 0 1 0, limit lower=-3.14159 upper=3.14159 effort=0.0 velocity=0.0

Commit message: N22

File: body.urdf (robot description, URDF)
Before this commit: robot robot, 3 links, 2 joints
Links:
- link BackLeg: geometry collision box size=0.2 1.0 0.2; visual box size=0.2 1.0 0.2
- link FrontLeg: geometry collision box size=0.2 1.0 0.2; visual box size=0.2 1.0 0.2
Joints:
- joint Torso_BackLeg: origin xyz=1 0 1 rpy=0 0 0 -> xyz=0.0 -0.5 1.0 rpy=0 0 0
- joint Torso_FrontLeg: origin xyz=2 0 1 rpy=0 0 0 -> xyz=0.0 0.5 1.0 rpy=0 0 0

Commit message: N44

File: body.urdf (robot description, URDF)
Before this commit: robot robot, 3 links, 2 joints
Links:
- added link BackLowerLeg, mass 1; collision box size=0.2 0.2 1.0; visual box size=0.2 0.2 1.0
- added link FrontLowerLeg, mass 1; collision box size=0.2 0.2 1.0; visual box size=0.2 0.2 1.0
- added link LeftLeg, mass 1; collision box size=1.0 0.2 0.2; visual box size=1.0 0.2 0.2
- added link LeftLowerLeg, mass 1; collision box size=0.2 0.2 1.0; visual box size=0.2 0.2 1.0
- added link RightLeg, mass 1; collision box size=1.0 0.2 0.2; visual box size=1.0 0.2 0.2
- added link RightLowerLeg, mass 1; collision box size=0.2 0.2 1.0; visual box size=0.2 0.2 1.0
- link Torso: geometry collision box size=1.0 1.0 1.0; visual box size=1.0 1.0 1.0
Joints:
- added joint BackLeg_BackLowerLeg: type revolute, parent BackLeg, child BackLowerLeg, origin xyz=0.0 -1.0 0.0 rpy=0 0 0, axis 1 0 0, limit lower=-3.14159 upper=3.14159 effort=0.0 velocity=0.0
- added joint FrontLeg_FrontLowerLeg: type revolute, parent FrontLeg, child FrontLowerLeg, origin xyz=0.0 1.0 0.0 rpy=0 0 0, axis 1 0 0, limit lower=-3.14159 upper=3.14159 effort=0.0 velocity=0.0
- added joint LeftLeg_LeftLowerLeg: type revolute, parent LeftLeg, child LeftLowerLeg, origin xyz=-1.0 0.0 0.0 rpy=0 0 0, axis 0 1 0, limit lower=-3.14159 upper=3.14159 effort=0.0 velocity=0.0
- added joint RightLeg_RightLowerLeg: type revolute, parent RightLeg, child RightLowerLeg, origin xyz=1.0 0.0 0.0 rpy=0 0 0, axis 0 1 0, limit lower=-3.14159 upper=3.14159 effort=0.0 velocity=0.0
- added joint Torso_LeftLeg: type revolute, parent Torso, child LeftLeg, origin xyz=-0.5 0.0 1.0 rpy=0 0 0, axis 0 1 0, limit lower=-3.14159 upper=3.14159 effort=0.0 velocity=0.0
- added joint Torso_RightLeg: type revolute, parent Torso, child RightLeg, origin xyz=0.5 0.0 1.0 rpy=0 0 0, axis 0 1 0, limit lower=-3.14159 upper=3.14159 effort=0.0 velocity=0.0
